File: hardware/outputdriver.sch (KiCad schematic (older format))
At the start: 22 parts, among them P3 COLUMNS, P4 ROWS, Q1 2N7000, Q10 2N7000, Q11 2N7000, Q12 2N7000, Q13 2N7000, Q14 2N7000, Q15 2N7000, Q16 2N7000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

Commit message: Beginning of PCB layout.
Parts:
- P3, P4: footprint (none) -> SIL-10
- Q1, Q10, Q11, Q12, Q13, Q14, Q15, Q16, Q17, Q18, Q19, Q2, Q20, Q3, Q4, Q5, Q6, Q7, Q8, Q9: footprint (none) -> TO92
Changed lines of the file:
@@
-EESchema Schematic File Version 2  date Thu 10 May 2012 01:29:50 BST
+EESchema Schematic File Version 2  date Tue 19 Jun 2012 03:11:31 BST
 LIBS:power
 LIBS:device
@@
 Sheet 2 2
 Title "Wordclock"
-Date "10 may 2012"
-Rev "1"
+Date "19 jun 2012"
+Rev "A"
 Comp "David Robertson"
-Comment1 ""
+Comment1 "http://davidr.me/"
 Comment2 ""
 Comment3 ""
@@
 P 6050 6700
 F 0 "#PWR015" H 6050 6790 20  0001 C CNN
-F 1 "+5V" H 6050 6790 30  0000 C CNN
+F 1 "+5V" H 6050 6850 30  0000 C CNN
 	1    6050 6700
 	-1   0    0    1
@@
 F 0 "Q11" H 6360 1270 60  0000 R CNN
 F 1 "2N7000" H 6360 950 60  0000 R CNN
+F 2 "TO92" H 6350 1100 60  0001 C CNN
 	1    6350 1100
 	-1   0    0    -1
@@
 F 0 "Q12" H 6360 1870 60  0000 R CNN
 F 1 "2N7000" H 6360 1550 60  0000 R CNN
+F 2 "TO92" H 6350 1700 60  0001 C CNN
 	1    6350 1700
 	-1   0    0    -1
@@
 F 0 "Q13" H 6360 2470 60  0000 R CNN
 F 1 "2N7000" H 6360 2150 60  0000 R CNN
+F 2 "TO92" H 6350 2300 60  0001 C CNN
 	1    6350 2300
 	-1   0    0    -1
@@
 F 0 "Q14" H 6360 3070 60  0000 R CNN
 F 1 "2N7000" H 6360 2750 60  0000 R CNN
+F 2 "TO92" H 6350 2900 60  0001 C CNN
 	1    6350 2900
 	-1   0    0    -1
@@
 F 0 "Q15" H 6360 3670 60  0000 R CNN
 F 1 "2N7000" H 6360 3350 60  0000 R CNN
+F 2 "TO92" H 6350 3500 60  0001 C CNN
 	1    6350 3500
 	-1   0    0    -1
@@
 F 0 "Q16" H 6360 4270 60  0000 R CNN
 F 1 "2N7000" H 6360 3950 60  0000 R CNN
+F 2 "TO92" H 6350 4100 60  0001 C CNN
 	1    6350 4100
 	-1   0    0    -1
@@
 F 0 "Q20" H 6360 6670 60  0000 R CNN
 F 1 "2N7000" H 6360 6350 60  0000 R CNN
+F 2 "TO92" H 6350 6500 60  0001 C CNN
 	1    6350 6500
 	-1   0    0    -1
@@
 F 0 "Q19" H 6360 6070 60  0000 R CNN
 F 1 "2N7000" H 6360 5750 60  0000 R CNN
+F 2 "TO92" H 6350 5900 60  0001 C CNN
 	1    6350 5900
 	-1   0    0    -1
@@
 F 0 "Q18" H 6360 5470 60  0000 R CNN
 F 1 "2N7000" H 6360 5150 60  0000 R CNN
+F 2 "TO92" H 6350 5300 60  0001 C CNN
 	1    6350 5300
 	-1   0    0    -1
@@
 F 0 "Q17" H 6360 4870 60  0000 R CNN
 F 1 "2N7000" H 6360 4550 60  0000 R CNN
+F 2 "TO92" H 6350 4700 60  0001 C CNN
 	1    6350 4700
 	-1   0    0    -1
@@
 F 0 "P4" V 8350 3900 60  0000 C CNN
 F 1 "ROWS" V 8450 3900 60  0000 C CNN
+F 2 "SIL-10" H 8400 3900 60  0001 C CNN
 	1    8400 3900
 	1    0    0    -1
@@
 F 0 "P3" V 3600 3500 60  0000 C CNN
 F 1 "COLUMNS" V 3700 3500 60  0000 C CNN
+F 2 "SIL-10" H 3650 3500 60  0001 C CNN
 	1    3650 3500
 	1    0    0    -1
@@
 F 0 "Q7" H 1510 4870 60  0000 R CNN
 F 1 "2N7000" H 1510 4550 60  0000 R CNN
+F 2 "TO92" H 1500 4700 60  0001 C CNN
 	1    1500 4700
 	-1   0    0    -1
@@
 F 0 "Q8" H 1510 5470 60  0000 R CNN
 F 1 "2N7000" H 1510 5150 60  0000 R CNN
+F 2 "TO92" H 1500 5300 60  0001 C CNN
 	1    1500 5300
 	-1   0    0    -1
@@
 F 0 "Q9" H 1510 6070 60  0000 R CNN
 F 1 "2N7000" H 1510 5750 60  0000 R CNN
+F 2 "TO92" H 1500 5900 60  0001 C CNN
 	1    1500 5900
 	-1   0    0    -1
@@
 F 0 "Q10" H 1510 6670 60  0000 R CNN
 F 1 "2N7000" H 1510 6350 60  0000 R CNN
+F 2 "TO92" H 1500 6500 60  0001 C CNN
 	1    1500 6500
 	-1   0    0    -1
@@
 F 0 "Q6" H 1510 4270 60  0000 R CNN
 F 1 "2N7000" H 1510 3950 60  0000 R CNN
+F 2 "TO92" H 1500 4100 60  0001 C CNN
 	1    1500 4100
 	-1   0    0    -1
@@
 F 0 "Q5" H 1510 3670 60  0000 R CNN
 F 1 "2N7000" H 1510 3350 60  0000 R CNN
+F 2 "TO92" H 1500 3500 60  0001 C CNN
 	1    1500 3500
 	-1   0    0    -1
@@
 F 0 "Q4" H 1510 3070 60  0000 R CNN
 F 1 "2N7000" H 1510 2750 60  0000 R CNN
+F 2 "TO92" H 1500 2900 60  0001 C CNN
 	1    1500 2900
 	-1   0    0    -1
@@
 F 0 "Q3" H 1510 2470 60  0000 R CNN
 F 1 "2N7000" H 1510 2150 60  0000 R CNN
+F 2 "TO92" H 1500 2300 60  0001 C CNN
 	1    1500 2300
 	-1   0    0    -1
@@
 F 0 "Q2" H 1510 1870 60  0000 R CNN
 F 1 "2N7000" H 1510 1550 60  0000 R CNN
+F 2 "TO92" H 1500 1700 60  0001 C CNN
 	1    1500 1700
 	-1   0    0    -1
@@
 F 0 "Q1" H 1510 1270 60  0000 R CNN
 F 1 "2N7000" H 1510 950 60  0000 R CNN
+F 2 "TO92" H 1500 1100 60  0001 C CNN
 	1    1500 1100
 	-1   0    0    -1
