File: hardware/wordclock.sch (KiCad schematic (older format))
At the start: 24 parts, among them K1 SERIAL, P1 ISP, P2 Vin, P5 Vin-alt, SW1 MINUTE, SW2 HOUR, U1 ATmega168, U2 DS1307, U3 7805, U4 4094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

Commit message: Finished PCB design, REV. A.
Parts:
- removed SW1: MINUTE, symbol SW_PUSH_SMALL
- removed SW2: HOUR, symbol SW_PUSH_SMALL
- added K2: CONN_3, symbol CONN_3
Connections:
- net B_HOUR: now also K2.3 (P3)
- net B_MIN: now also K2.2 (PM)
- net GND: now also K2.1 (P1)
Other:
- moved on the sheet: C6, C7, R3, R4
Changed lines of the file:
@@
-EESchema Schematic File Version 2  date Wed 11 Jul 2012 22:54:35 BST
+EESchema Schematic File Version 2  date Tue 17 Jul 2012 20:32:37 BST
 LIBS:power
 LIBS:device
@@
 Sheet 1 2
 Title "Wordclock"
-Date "11 jul 2012"
-Rev "1"
+Date "17 jul 2012"
+Rev "A"
 Comp "David Robertson"
-Comment1 ""
+Comment1 "http://davidr.me/projects/word-clock"
 Comment2 ""
 Comment3 ""
 Comment4 ""
 $EndDescr
-$Comp
-L SW_PUSH_SMALL SW2
-U 1 1 4FFDF2DD
-P 3450 5450
-F 0 "SW2" H 3600 5560 30  0000 C CNN
-F 1 "HOUR" H 3400 5350 30  0000 C CNN
-	1    3450 5450
-	1    0    0    -1
-$EndComp
-$Comp
-L CP1 C7
-U 1 1 4FFDF2DC
-P 2900 5550
-F 0 "C7" H 2950 5650 50  0000 L CNN
-F 1 "1uF" H 2950 5450 50  0000 L CNN
-	1    2900 5550
-	1    0    0    -1
-$EndComp
-Text Label 3000 5350 0    60   ~ 0
-B_HOUR
-$Comp
-L R R4
-U 1 1 4FFDF2DB
-P 2900 5100
-F 0 "R4" V 2980 5100 50  0000 C CNN
-F 1 "10K" V 2900 5100 50  0000 C CNN
-	1    2900 5100
-	1    0    0    -1
-$EndComp
-$Comp
-L GND #PWR01
-U 1 1 4FFDF2DA
-P 3550 5800
-F 0 "#PWR01" H 3550 5800 30  0001 C CNN
-F 1 "GND" H 3550 5730 30  0001 C CNN
-	1    3550 5800
-	1    0    0    -1
-$EndComp
-Wire Wire Line
-	3550 5800 3550 5550
-Wire Wire Line
-	2900 5350 3350 5350
-Wire Wire Line
-	2900 5750 3550 5750
-Connection ~ 3550 5750
-$Comp
-L +5V #PWR02
-U 1 1 4FFDF2D9
-P 2900 4850
-F 0 "#PWR02" H 2900 4940 20  0001 C CNN
-F 1 "+5V" H 2900 4940 30  0000 C CNN
-	1    2900 4850
-	1    0    0    -1
-$EndComp
-$Comp
-L +5V #PWR03
-U 1 1 4FFDF2C9
-P 2000 4850
-F 0 "#PWR03" H 2000 4940 20  0001 C CNN
-F 1 "+5V" H 2000 4940 30  0000 C CNN
-	1    2000 4850
-	1    0    0    -1
-$EndComp
-Connection ~ 2650 5750
-Wire Wire Line
-	2000 5750 2650 5750
-Wire Wire Line
-	2000 5350 2450 5350
+NoConn ~ 1300 2400
+NoConn ~ 1300 2200
+NoConn ~ 1300 1800
+NoConn ~ 3200 3100
+NoConn ~ 3200 3000
+NoConn ~ 3200 2900
+Wire Wire Line
+	6150 4100 6150 3950
+Wire Wire Line
+	2000 5200 2000 5550
+Wire Wire Line
+	2000 5550 1350 5550
+Wire Wire Line
+	2650 5550 2100 5550
+Wire Wire Line
+	1350 6000 1350 5950
 Connection ~ 4250 7450
 Wire Wire Line
@@
 Wire Wire Line
 	1350 6550 1550 6550
-Wire Wire Line
-	6150 3950 6150 4050
 Wire Wire Line
 	3200 1600 5400 1600
@@
 Connection ~ 4150 6750
 Wire Wire Line
-	2650 5800 2650 5550
-$Comp
-L GND #PWR04
+	2650 5950 2650 6000
+Wire Wire Line
+	2100 5550 2100 5200
+Wire Wire Line
+	1900 5350 1900 5200
+$Comp
+L GND #PWR01
+U 1 1 5005AE3A
+P 1900 5350
+F 0 "#PWR01" H 1900 5350 30  0001 C CNN
+F 1 "GND" H 1900 5280 30  0001 C CNN
+	1    1900 5350
+	1    0    0    -1
+$EndComp
+$Comp
+L CONN_3 K2
+U 1 1 5005AD69
+P 2000 4850
+F 0 "K2" V 1950 4850 50  0000 C CNN
+F 1 "CONN_3" V 2050 4850 40  0000 C CNN
+	1    2000 4850
+	0    -1   -1   0
+$EndComp
+$Comp
+L CP1 C7
+U 1 1 4FFDF2DC
+P 2650 5750
+F 0 "C7" H 2700 5850 50  0000 L CNN
+F 1 "1uF" H 2700 5650 50  0000 L CNN
+	1    2650 5750
+	1    0    0    -1
+$EndComp
+Text Label 2200 5550 0    60   ~ 0
+B_HOUR
+$Comp
+L R R4
+U 1 1 4FFDF2DB
+P 2650 5300
+F 0 "R4" V 2730 5300 50  0000 C CNN
+F 1 "10K" V 2650 5300 50  0000 C CNN
+	1    2650 5300
+	1    0    0    -1
+$EndComp
+$Comp
+L GND #PWR02
+U 1 1 4FFDF2DA
+P 2650 6000
+F 0 "#PWR02" H 2650 6000 30  0001 C CNN
+F 1 "GND" H 2650 5930 30  0001 C CNN
+	1    2650 6000
+	1    0    0    -1
+$EndComp
+$Comp
+L +5V #PWR03
+U 1 1 4FFDF2D9
+P 2650 5050
+F 0 "#PWR03" H 2650 5140 20  0001 C CNN
+F 1 "+5V" H 2650 5140 30  0000 C CNN
+	1    2650 5050
+	1    0    0    -1
+$EndComp
+$Comp
+L +5V #PWR04
+U 1 1 4FFDF2C9
+P 1350 5050
+F 0 "#PWR04" H 1350 5140 20  0001 C CNN
+F 1 "+5V" H 1350 5140 30  0000 C CNN
+	1    1350 5050
+	1    0    0    -1
+$EndComp
+$Comp
+L GND #PWR05
 U 1 1 4FFDF297
-P 2650 5800
-F 0 "#PWR04" H 2650 5800 30  0001 C CNN
-F 1 "GND" H 2650 5730 30  0001 C CNN
-	1    2650 5800
+P 1350 6000
+F 0 "#PWR05" H 1350 6000 30  0001 C CNN
+F 1 "GND" H 1350 5930 30  0001 C CNN
+	1    1350 6000
 	1    0    0    -1
 $EndComp
@@
 L R R3
 U 1 1 4FFDF27A
-P 2000 5100
-F 0 "R3" V 2080 5100 50  0000 C CNN
-F 1 "10K" V 2000 5100 50  0000 C CNN
-	1    2000 5100
+P 1350 5300
+F 0 "R3" V 1430 5300 50  0000 C CNN
+F 1 "10K" V 1350 5300 50  0000 C CNN
+	1    1350 5300
 	1    0    0    -1
 $EndComp
@@
 Text Label 3200 2600 0    60   ~ 0
 B_MIN
-Text Label 2100 5350 0    60   ~ 0
+Text Label 1800 5550 2    60   ~ 0
 B_MIN
 $Comp
 L CP1 C?
 U 1 1 4FFDF1A6
-P 2000 5550
+P 1350 5750
 AR Path="/4FFDF19E" Ref="C?"  Part="1"
 AR Path="/4FFDF1A6" Ref="C6"  Part="1"
-F 0 "C6" H 2050 5650 50  0000 L CNN
-F 1 "1uF" H 2050 5450 50  0000 L CNN
-	1    2000 5550
-	1    0    0    -1
-$EndComp
-$Comp
-L SW_PUSH_SMALL SW?
-U 1 1 4FFDF13E
-P 2550 5450
-AR Path="/4FFDF125" Ref="SW?"  Part="1"
-AR Path="/4FFDF13E" Ref="SW1"  Part="1"
-F 0 "SW1" H 2700 5560 30  0000 C CNN
-F 1 "MINUTE" H 2500 5350 30  0000 C CNN
-	1    2550 5450
+F 0 "C6" H 1400 5850 50  0000 L CNN
+F 1 "1uF" H 1400 5650 50  0000 L CNN
+	1    1350 5750
 	1    0    0    -1
 $EndComp
@@
 Vin
 $Comp
-L +5V #PWR05
+L +5V #PWR06
 U 1 1 4FDFF8A7
 P 2250 7500
-F 0 "#PWR05" H 2250 7590 20  0001 C CNN
+F 0 "#PWR06" H 2250 7590 20  0001 C CNN
 F 1 "+5V" H 2250 7650 30  0000 C CNN
 	1    2250 7500
@@
 Voltage Regulator
 $Comp
-L GND #PWR06
+L GND #PWR07
 U 1 1 4FAB0608
 P 1400 7250
-F 0 "#PWR06" H 1400 7250 30  0001 C CNN
+F 0 "#PWR07" H 1400 7250 30  0001 C CNN
 F 1 "GND" H 1400 7180 30  0001 C CNN
 	1    1400 7250
@@
 $EndComp
 $Comp
-L +5V #PWR07
+L +5V #PWR08
 U 1 1 4FAB05EC
 P 5950 6650
-F 0 "#PWR07" H 5950 6740 20  0001 C CNN
+F 0 "#PWR08" H 5950 6740 20  0001 C CNN
 F 1 "+5V" H 5950 6740 30  0000 C CNN
 	1    5950 6650
@@
 $EndComp
 $Comp
-L GND #PWR08
+L GND #PWR09
 U 1 1 4FAB05E1
 P 5950 7550
-F 0 "#PWR08" H 5950 7550 30  0001 C CNN
+F 0 "#PWR09" H 5950 7550 30  0001 C CNN
 F 1 "GND" H 5950 7480 30  0001 C CNN
 	1    5950 7550
@@
 $EndComp
 $Comp
-L GND #PWR09
+L GND #PWR010
 U 1 1 4FAB056E
 P 3550 2550
-F 0 "#PWR09" H 3550 2550 30  0001 C CNN
+F 0 "#PWR010" H 3550 2550 30  0001 C CNN
 F 1 "GND" H 3550 2480 30  0001 C CNN
 	1    3550 2550
@@
 	1    0    0    -1
 $EndComp
-NoConn ~ 1300 1800
-NoConn ~ 3200 3100
-NoConn ~ 3200 3000
-NoConn ~ 3200 2900
 Text Notes 3350 6400 2    60   ~ 0
 RTC
@@
 $EndComp
 $Comp
-L +5V #PWR010
+L +5V #PWR011
 U 1 1 4FAAF7B7
 P 4100 4050
-F 0 "#PWR010" H 4100 4140 20  0001 C CNN
+F 0 "#PWR011" H 4100 4140 20  0001 C CNN
 F 1 "+5V" H 4100 4200 30  0000 C CNN
 	1    4100 4050
 	1    0    0    -1
 $EndComp
-NoConn ~ 1300 2200
-NoConn ~ 1300 2400
-$Comp
-L GND #PWR011
+$Comp
+L GND #PWR012
 U 1 1 4FAAF757
 P 4100 4450
-F 0 "#PWR011" H 4100 4450 30  0001 C CNN
+F 0 "#PWR012" H 4100 4450 30  0001 C CNN
 F 1 "GND" H 4100 4380 30  0001 C CNN
 	1    4100 4450
@@
 NoConn ~ 6900 2100
 $Comp
-L +5V #PWR012
+L +5V #PWR013
 U 1 1 4FAAF0EA
 P 7000 1500
-F 0 "#PWR012" H 7000 1590 20  0001 C CNN
+F 0 "#PWR013" H 7000 1590 20  0001 C CNN
 F 1 "+5V" H 7000 1650 30  0000 C CNN
 	1    7000 1500
@@
 $EndComp
 $Comp
-L GND #PWR013
+L GND #PWR014
 U 1 1 4FAAF091
 P 5400 2250
-F 0 "#PWR013" H 5400 2250 30  0001 C CNN
+F 0 "#PWR014" H 5400 2250 30  0001 C CNN
 F 1 "GND" H 5400 2180 30  0001 C CNN
 	1    5400 2250
@@
 1Hz
 $Comp
-L +5V #PWR014
+L +5V #PWR015
 U 1 1 4FAAEF1A
 P 3100 6550
-F 0 "#PWR014" H 3100 6640 20  0001 C CNN
+F 0 "#PWR015" H 3100 6640 20  0001 C CNN
 F 1 "+5V" H 3100 6640 30  0000 C CNN
 	1    3100 6550
@@
 $EndComp
 $Comp
-L +5V #PWR015
+L +5V #PWR016
 U 1 1 4FAAEF0F
 P 2200 1150
-F 0 "#PWR015" H 2200 1240 20  0001 C CNN
+F 0 "#PWR016" H 2200 1240 20  0001 C CNN
 F 1 "+5V" H 2200 1300 30  0000 C CNN
 	1    2200 1150
@@
 $EndComp
 $Comp
-L +5V #PWR016
+L +5V #PWR017
 U 1 1 4FAAEF01
 P 6150 2650
-F 0 "#PWR016" H 6150 2740 20  0001 C CNN
+F 0 "#PWR017" H 6150 2740 20  0001 C CNN
 F 1 "+5V" H 6250 2700 30  0000 C CNN
 	1    6150 2650
@@
 $EndComp
 $Comp
-L GND #PWR017
+L GND #PWR018
 U 1 1 4FAAEED9
-P 6150 4050
-F 0 "#PWR017" H 6150 4050 30  0001 C CNN
-F 1 "GND" H 6150 3980 30  0001 C CNN
-	1    6150 4050
+P 6150 4100
+F 0 "#PWR018" H 6150 4100 30  0001 C CNN
+F 1 "GND" H 6150 4030 30  0001 C CNN
+	1    6150 4100
 	1    0    0    -1
 $EndComp
@@
 $EndComp
 $Comp
-L GND #PWR018
+L GND #PWR019
 U 1 1 4FAAEEA0
 P 2200 4150
-F 0 "#PWR018" H 2200 4150 30  0001 C CNN
+F 0 "#PWR019" H 2200 4150 30  0001 C CNN
 F 1 "GND" H 2200 4080 30  0001 C CNN
 	1    2200 4150
@@
 $EndComp
 $Comp
-L GND #PWR019
+L GND #PWR020
 U 1 1 4FAAEE8C
 P 1550 6900
-F 0 "#PWR019" H 1550 6900 30  0001 C CNN
+F 0 "#PWR020" H 1550 6900 30  0001 C CNN
 F 1 "GND" H 1550 6830 30  0001 C CNN
 	1    1550 6900
